File: hw/launch-it.kicad_sch (KiCad schematic)
At the start: 100 parts, among them J1 SWD, M1 Motor_DC, Q1 PJA3401A, Q2 AO3400A, U1 STM32F030F4, U2 MCP1603, U3 IS31FL3731-SA, U4 CAP1203-1-SN

Commit message: updated CR2032 PN and minimal layout updates
Parts:
- BT2: DK_PN 1908-CR2032-ND -> 343-BAT-HLD-003-SMT-ND
Changed lines of the file:
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@@
 			)
 		)
-		(property "DK_PN" "1908-CR2032-ND "
+		(property "DK_PN" "343-BAT-HLD-003-SMT-ND "
 			(at 40.64 67.31 0)
 			(effects
